Commit message: Implemented variables

File: description/robot_core.xacro (robot description, xacro)
@@ -2,4 +2,16 @@
 <robot xmlns:xacro="http://www.ros.org/wiki/xacro">
     <xacro:include filename='inertial_macros.xacro'/>
+    <xacro:property name="chassis_length" value="0.4953"/>
+    <xacro:property name="chassis_width" value="0.4064"/>
+    <xacro:property name="chassis_height" value="0.0635"/>
+    <xacro:property name="chassis_mass" value="1.0"/>
+    <xacro:property name="wheel_radius" value="0.130"/>
+    <xacro:property name="wheel_thickness" value="0.085"/>
+    <xacro:property name="wheel_mass" value="0.05"/>
+    <xacro:property name="hub_length" value="0.4445"/>
+    <xacro:property name="hub_radius" value="0.0254"/>
+    <!--ROS2 x and y conventions-->
+    <xacro:property name="botcnt2whlcnt_x" value="0.19685"/>
+    <xacro:property name="botcnt2whlcnt_y" value="0.22225"/>
     <material name="white">
         <color rgba="1 1 1 1"/>
@@ -18,30 +30,26 @@
     </link>
     <!-- CHASSIS -->
-    <!-- Bottom plate .125" not included -->
-    <!--
-        Weight of entire chassis including hubs and bottom
-        in kg is:
-    -->
+    <!-- Bottom plate .125" not included in robot model-->
     <joint name="chassis_joint" type="fixed">
         <parent link="base_link"/>
         <child link="chassis"/>
-        <origin xyz="-0.24765 0 -0.03175"/>
+        <origin xyz="${-chassis_length/2} 0 ${-chassis_height/2}"/>
     </joint>
     <link name="chassis">
         <visual>
-            <origin xyz="0.24765 0 0.03175"/>
-            <geometry>
-                <box size=".4953 .4064 .0635"/>
+            <origin xyz="${chassis_length/2} 0 ${chassis_height/2}"/>
+            <geometry>
+                <box size="${chassis_length} ${chassis_width} ${chassis_height}"/>
             </geometry>
             <material name="white"/>
         </visual>
         <collision>
-            <origin xyz="0.24765 0 0.03175"/>
-            <geometry>
-                <box size=".4953 .4064 .0635"/>
-            </geometry>
-        </collision>
-        <xacro:inertial_box mass="12" x="0.4953" y="0.4046" z="0.0635">
-            <origin xyz="0.24765 0 0.03175" rpy="0 0 0"/>
+            <origin xyz="${chassis_length/2} 0 ${chassis_height/2}"/>
+            <geometry>
+                <box size="${chassis_length} ${chassis_width} ${chassis_height}"/>
+            </geometry>
+        </collision>
+        <xacro:inertial_box mass="${chassis_mass}" x="${chassis_length}" y="${chassis_width}" z="${chassis_height}">
+            <origin xyz="${chassis_length/2} 0 ${chassis_height/2}" rpy="0 0 0"/>
         </xacro:inertial_box>
     </link>
@@ -53,5 +61,5 @@
         <parent link="base_link"/>
         <child link="front_hub"/>
-        <origin xyz="0.19685 0 0" rpy="${pi/2} 0 0"/>
+        <origin xyz="${botcnt2whlcnt_x} 0 0" rpy="${pi/2} 0 0"/>
     </joint>
     <link name="front_hub">
@@ -59,5 +67,5 @@
             <origin xyz="0 0 0"/>
             <geometry>
-                <cylinder radius="0.0254" length="0.4445"/>
+                <cylinder radius="${hub_radius}" length="${hub_length}"/>
             </geometry>
             <material name="white"/>
@@ -71,5 +79,5 @@
         <parent link="base_link"/>
         <child link="back_hub"/>
-        <origin xyz="-0.19685 0 0" rpy="${pi/2} 0 0"/>
+        <origin xyz="${-botcnt2whlcnt_x} 0 0" rpy="${pi/2} 0 0"/>
     </joint>
     <link name="back_hub">
@@ -77,5 +85,5 @@
             <origin xyz="0 0 0"/>
             <geometry>
-                <cylinder radius="0.0254" length="0.4445"/>
+                <cylinder radius="${hub_radius}" length="${hub_length}"/>
             </geometry>
             <material name="white"/>
@@ -86,27 +94,26 @@
     </gazebo>
     <!-- FRONT LEFT WHEEL LINK -->
-    <!-- Weight of each wheel: kg-->
     <joint name="front_left_wheel_joint" type="continuous">
         <parent link="base_link"/>
         <child link="front_left_wheel"/>
-        <origin xyz="0.19685 0.22225 0" rpy="-${pi/2} 0 0"/>
+        <origin xyz="${botcnt2whlcnt_x} ${botcnt2whlcnt_y} 0" rpy="-${pi/2} 0 0"/>
         <axis xyz="0 0 1"/>
     </joint>
     <link name="front_left_wheel">
         <visual>
-            <origin xyz="0 0 0.0425"/>
-            <geometry>
-                <cylinder radius="0.130" length=".085"/>
-            </geometry>
-            <material name="blue"/>
-        </visual>
-        <collision>
-            <origin xyz="0 0 0.0425"/>
-            <geometry>
-                <cylinder radius="0.130" length=".085"/>
-            </geometry>
-        </collision>
-        <xacro:inertial_cylinder mass="2" length=".085" radius="0.130">
-            <origin xyz="0 0 0.0425" rpy="0 0 0"/>
+            <origin xyz="0 0 ${wheel_thickness/2}"/>
+            <geometry>
+                <cylinder radius="${wheel_radius}" length="${wheel_thickness}"/>
+            </geometry>
+            <material name="blue"/>
+        </visual>
+        <collision>
+            <origin xyz="0 0 ${wheel_thickness/2}"/>
+            <geometry>
+                <cylinder radius="${wheel_radius}" length="${wheel_thickness}"/>
+            </geometry>
+        </collision>
+        <xacro:inertial_cylinder mass="${wheel_mass}" length="${wheel_thickness}" radius="${wheel_radius}">
+            <origin xyz="0 0 ${wheel_thickness/2}" rpy="0 0 0"/>
         </xacro:inertial_cylinder>
     </link>
@@ -118,23 +125,23 @@
         <parent link="base_link"/>
         <child link="back_left_wheel"/>
-        <origin xyz="-0.19685 0.22225 0" rpy="-${pi/2} 0 0"/>
+        <origin xyz="${-botcnt2whlcnt_x} ${botcnt2whlcnt_y} 0" rpy="-${pi/2} 0 0"/>
         <axis xyz="0 0 1"/>
     </joint>
     <link name="back_left_wheel">
         <visual>
-            <origin xyz="0 0 0.0425"/>
-            <geometry>
-                <cylinder radius="0.130" length=".085"/>
-            </geometry>
-            <material name="blue"/>
-        </visual>
-        <collision>
-            <origin xyz="0 0 0.0425"/>
-            <geometry>
-                <cylinder radius="0.130" length=".085"/>
-            </geometry>
-        </collision>
-        <xacro:inertial_cylinder mass="2" length=".085" radius="0.130">
-            <origin xyz="0 0 0.0425" rpy="0 0 0"/>
+            <origin xyz="0 0 ${wheel_thickness/2}"/>
+            <geometry>
+                <cylinder radius="${wheel_radius}" length="${wheel_thickness}"/>
+            </geometry>
+            <material name="blue"/>
+        </visual>
+        <collision>
+            <origin xyz="0 0 ${wheel_thickness/2}"/>
+            <geometry>
+                <cylinder radius="${wheel_radius}" length="${wheel_thickness}"/>
+            </geometry>
+        </collision>
+        <xacro:inertial_cylinder mass="${wheel_mass}" length="${wheel_thickness}" radius="${wheel_radius}">
+            <origin xyz="0 0 ${wheel_thickness/2}" rpy="0 0 0"/>
         </xacro:inertial_cylinder>
     </link>
@@ -146,23 +153,23 @@
         <parent link="base_link"/>
         <child link="front_right_wheel"/>
-        <origin xyz="0.19685 -0.22225 0" rpy="${pi/2} 0 0"/>
+        <origin xyz="${botcnt2whlcnt_x} ${-botcnt2whlcnt_y} 0" rpy="${pi/2} 0 0"/>
         <axis xyz="0 0 -1"/>
     </joint>
     <link name="front_right_wheel">
         <visual>
-            <origin xyz="0 0 0.0425"/>
-            <geometry>
-                <cylinder radius="0.130" length=".085"/>
-            </geometry>
-            <material name="blue"/>
-        </visual>
-        <collision>
-            <origin xyz="0 0 0.0425"/>
-            <geometry>
-                <cylinder radius="0.130" length=".085"/>
-            </geometry>
-        </collision>
-        <xacro:inertial_cylinder mass="2" length=".085" radius="0.130">
-            <origin xyz="0 0 0.0425" rpy="0 0 0"/>
+            <origin xyz="0 0 ${wheel_thickness/2}"/>
+            <geometry>
+                <cylinder radius="${wheel_radius}" length="${wheel_thickness}"/>
+            </geometry>
+            <material name="blue"/>
+        </visual>
+        <collision>
+            <origin xyz="0 0 ${wheel_thickness/2}"/>
+            <geometry>
+                <cylinder radius="${wheel_radius}" length="${wheel_thickness}"/>
+            </geometry>
+        </collision>
+        <xacro:inertial_cylinder mass="${wheel_mass}" length="${wheel_thickness}" radius="${wheel_radius}">
+            <origin xyz="0 0 ${wheel_thickness/2}" rpy="0 0 0"/>
         </xacro:inertial_cylinder>
     </link>
@@ -174,23 +181,23 @@
         <parent link="base_link"/>
         <child link="back_right_wheel"/>
-        <origin xyz="-0.19685 -0.22225 0" rpy="${pi/2} 0 0"/>
+        <origin xyz="${-botcnt2whlcnt_x} ${-botcnt2whlcnt_y} 0" rpy="${pi/2} 0 0"/>
         <axis xyz="0 0 -1"/>
     </joint>
     <link name="back_right_wheel">
         <visual>
-            <origin xyz="0 0 0.0425"/>
-            <geometry>
-                <cylinder radius="0.130" length=".085"/>
-            </geometry>
-            <material name="blue"/>
-        </visual>
-        <collision>
-            <origin xyz="0 0 0.0425"/>
-            <geometry>
-                <cylinder radius="0.130" length=".085"/>
-            </geometry>
-        </collision>
-        <xacro:inertial_cylinder mass="2" length=".085" radius="0.130">
-            <origin xyz="0 0 0.0425" rpy="0 0 0"/>
+            <origin xyz="0 0 ${wheel_thickness/2}"/>
+            <geometry>
+                <cylinder radius="${wheel_radius}" length="${wheel_thickness}"/>
+            </geometry>
+            <material name="blue"/>
+        </visual>
+        <collision>
+            <origin xyz="0 0 ${wheel_thickness/2}"/>
+            <geometry>
+                <cylinder radius="${wheel_radius}" length="${wheel_thickness}"/>
+            </geometry>
+        </collision>
+        <xacro:inertial_cylinder mass="${wheel_mass}" length="${wheel_thickness}" radius="${wheel_radius}">
+            <origin xyz="0 0 ${wheel_thickness/2}" rpy="0 0 0"/>
         </xacro:inertial_cylinder>
     </link>

Commit message: Implemented proper snake case to variables

File: description/robot_core.xacro (robot description, xacro)
@@ -12,6 +12,6 @@
     <xacro:property name="hub_radius" value="0.0254"/>
     <!--ROS2 x and y conventions-->
-    <xacro:property name="botcnt2whlcnt_x" value="0.19685"/>
-    <xacro:property name="botcnt2whlcnt_y" value="0.22225"/>
+    <xacro:property name="bot_center_to_wheel_center_x" value="0.19685"/>
+    <xacro:property name="bot_center_to_wheel_center_y" value="0.22225"/>
     <material name="white">
         <color rgba="1 1 1 1"/>
@@ -61,5 +61,5 @@
         <parent link="base_link"/>
         <child link="front_hub"/>
-        <origin xyz="${botcnt2whlcnt_x} 0 0" rpy="${pi/2} 0 0"/>
+        <origin xyz="${bot_center_to_wheel_center_x} 0 0" rpy="${pi/2} 0 0"/>
     </joint>
     <link name="front_hub">
@@ -79,5 +79,5 @@
         <parent link="base_link"/>
         <child link="back_hub"/>
-        <origin xyz="${-botcnt2whlcnt_x} 0 0" rpy="${pi/2} 0 0"/>
+        <origin xyz="${-bot_center_to_wheel_center_x} 0 0" rpy="${pi/2} 0 0"/>
     </joint>
     <link name="back_hub">
@@ -97,5 +97,5 @@
         <parent link="base_link"/>
         <child link="front_left_wheel"/>
-        <origin xyz="${botcnt2whlcnt_x} ${botcnt2whlcnt_y} 0" rpy="-${pi/2} 0 0"/>
+        <origin xyz="${bot_center_to_wheel_center_x} ${bot_center_to_wheel_center_y} 0" rpy="-${pi/2} 0 0"/>
         <axis xyz="0 0 1"/>
     </joint>
@@ -125,5 +125,5 @@
         <parent link="base_link"/>
         <child link="back_left_wheel"/>
-        <origin xyz="${-botcnt2whlcnt_x} ${botcnt2whlcnt_y} 0" rpy="-${pi/2} 0 0"/>
+        <origin xyz="${-bot_center_to_wheel_center_x} ${bot_center_to_wheel_center_y} 0" rpy="-${pi/2} 0 0"/>
         <axis xyz="0 0 1"/>
     </joint>
@@ -153,5 +153,5 @@
         <parent link="base_link"/>
         <child link="front_right_wheel"/>
-        <origin xyz="${botcnt2whlcnt_x} ${-botcnt2whlcnt_y} 0" rpy="${pi/2} 0 0"/>
+        <origin xyz="${bot_center_to_wheel_center_x} ${-bot_center_to_wheel_center_y} 0" rpy="${pi/2} 0 0"/>
         <axis xyz="0 0 -1"/>
     </joint>
@@ -181,5 +181,5 @@
         <parent link="base_link"/>
         <child link="back_right_wheel"/>
-        <origin xyz="${-botcnt2whlcnt_x} ${-botcnt2whlcnt_y} 0" rpy="${pi/2} 0 0"/>
+        <origin xyz="${-bot_center_to_wheel_center_x} ${-bot_center_to_wheel_center_y} 0" rpy="${pi/2} 0 0"/>
         <axis xyz="0 0 -1"/>
     </joint>

Commit message: Added macros to simplify wheel declarations

File: description/robot_core.xacro (robot description, xacro)
@@ -57,4 +57,5 @@
         <material>Gazebo/White</material>
     </gazebo>
+    <!-- HUBS -->
     <!-- FRONT HUB-->
     <joint name="front_hub_joint" type="fixed">
@@ -93,115 +94,20 @@
         <material>Gazebo/White</material>
     </gazebo>
+    <!-- WHEELS -->
     <!-- FRONT LEFT WHEEL LINK -->
-    <joint name="front_left_wheel_joint" type="continuous">
-        <parent link="base_link"/>
-        <child link="front_left_wheel"/>
-        <origin xyz="${bot_center_to_wheel_center_x} ${bot_center_to_wheel_center_y} 0" rpy="-${pi/2} 0 0"/>
-        <axis xyz="0 0 1"/>
-    </joint>
-    <link name="front_left_wheel">
-        <visual>
-            <origin xyz="0 0 ${wheel_thickness/2}"/>
-            <geometry>
-                <cylinder radius="${wheel_radius}" length="${wheel_thickness}"/>
-            </geometry>
-            <material name="blue"/>
-        </visual>
-        <collision>
-            <origin xyz="0 0 ${wheel_thickness/2}"/>
-            <geometry>
-                <cylinder radius="${wheel_radius}" length="${wheel_thickness}"/>
-            </geometry>
-        </collision>
-        <xacro:inertial_cylinder mass="${wheel_mass}" length="${wheel_thickness}" radius="${wheel_radius}">
-            <origin xyz="0 0 ${wheel_thickness/2}" rpy="0 0 0"/>
-        </xacro:inertial_cylinder>
-    </link>
-    <gazebo reference="front_left_wheel">
-        <material>Gazebo/Blue</material>
-    </gazebo>
+    <xacro:wheel_joint position="front_left" bot_center_to_wheel_center_x="${bot_center_to_wheel_center_x}" bot_center_to_wheel_center_y="${bot_center_to_wheel_center_y}"/>
+    <!-- FRONT LEFT WHEEL JOINT -->
+    <xacro:wheel position="front_left" radius="${wheel_radius}" thickness="${wheel_thickness}" mass="${wheel_mass}"/>
     <!-- BACK LEFT WHEEL LINK -->
-    <joint name="back_left_wheel_joint" type="continuous">
-        <parent link="base_link"/>
-        <child link="back_left_wheel"/>
-        <origin xyz="${-bot_center_to_wheel_center_x} ${bot_center_to_wheel_center_y} 0" rpy="-${pi/2} 0 0"/>
-        <axis xyz="0 0 1"/>
-    </joint>
-    <link name="back_left_wheel">
-        <visual>
-            <origin xyz="0 0 ${wheel_thickness/2}"/>
-            <geometry>
-                <cylinder radius="${wheel_radius}" length="${wheel_thickness}"/>
-            </geometry>
-            <material name="blue"/>
-        </visual>
-        <collision>
-            <origin xyz="0 0 ${wheel_thickness/2}"/>
-            <geometry>
-                <cylinder radius="${wheel_radius}" length="${wheel_thickness}"/>
-            </geometry>
-        </collision>
-        <xacro:inertial_cylinder mass="${wheel_mass}" length="${wheel_thickness}" radius="${wheel_radius}">
-            <origin xyz="0 0 ${wheel_thickness/2}" rpy="0 0 0"/>
-        </xacro:inertial_cylinder>
-    </link>
-    <gazebo reference="back_left_wheel">
-        <material>Gazebo/Blue</material>
-    </gazebo>
+    <xacro:wheel_joint position="back_left" bot_center_to_wheel_center_x="${bot_center_to_wheel_center_x}" bot_center_to_wheel_center_y="${bot_center_to_wheel_center_y}"/>
+    <!-- BACK LEFT WHEEL JOINT -->
+    <xacro:wheel position="back_left" radius="${wheel_radius}" thickness="${wheel_thickness}" mass="${wheel_mass}"/>
     <!-- FRONT RIGHT WHEEL LINK -->
-    <joint name="front_right_wheel_joint" type="continuous">
-        <parent link="base_link"/>
-        <child link="front_right_wheel"/>
-        <origin xyz="${bot_center_to_wheel_center_x} ${-bot_center_to_wheel_center_y} 0" rpy="${pi/2} 0 0"/>
-        <axis xyz="0 0 -1"/>
-    </joint>
-    <link name="front_right_wheel">
-        <visual>
-            <origin xyz="0 0 ${wheel_thickness/2}"/>
-            <geometry>
-                <cylinder radius="${wheel_radius}" length="${wheel_thickness}"/>
-            </geometry>
-            <material name="blue"/>
-        </visual>
-        <collision>
-            <origin xyz="0 0 ${wheel_thickness/2}"/>
-            <geometry>
-                <cylinder radius="${wheel_radius}" length="${wheel_thickness}"/>
-            </geometry>
-        </collision>
-        <xacro:inertial_cylinder mass="${wheel_mass}" length="${wheel_thickness}" radius="${wheel_radius}">
-            <origin xyz="0 0 ${wheel_thickness/2}" rpy="0 0 0"/>
-        </xacro:inertial_cylinder>
-    </link>
-    <gazebo reference="front_right_wheel">
-        <material>Gazebo/Blue</material>
-    </gazebo>
+    <xacro:wheel_joint position="front_right" bot_center_to_wheel_center_x="${bot_center_to_wheel_center_x}" bot_center_to_wheel_center_y="${bot_center_to_wheel_center_y}"/>
+    <!-- FRONT RIGHT WHEEL JOINT -->
+    <xacro:wheel position="front_right" radius="${wheel_radius}" thickness="${wheel_thickness}" mass="${wheel_mass}"/>
     <!-- BACK RIGHT WHEEL LINK -->
-    <joint name="back_right_wheel_joint" type="continuous">
-        <parent link="base_link"/>
-        <child link="back_right_wheel"/>
-        <origin xyz="${-bot_center_to_wheel_center_x} ${-bot_center_to_wheel_center_y} 0" rpy="${pi/2} 0 0"/>
-        <axis xyz="0 0 -1"/>
-    </joint>
-    <link name="back_right_wheel">
-        <visual>
-            <origin xyz="0 0 ${wheel_thickness/2}"/>
-            <geometry>
-                <cylinder radius="${wheel_radius}" length="${wheel_thickness}"/>
-            </geometry>
-            <material name="blue"/>
-        </visual>
-        <collision>
-            <origin xyz="0 0 ${wheel_thickness/2}"/>
-            <geometry>
-                <cylinder radius="${wheel_radius}" length="${wheel_thickness}"/>
-            </geometry>
-        </collision>
-        <xacro:inertial_cylinder mass="${wheel_mass}" length="${wheel_thickness}" radius="${wheel_radius}">
-            <origin xyz="0 0 ${wheel_thickness/2}" rpy="0 0 0"/>
-        </xacro:inertial_cylinder>
-    </link>
-    <gazebo reference="back_right_wheel">
-        <material>Gazebo/Blue</material>
-    </gazebo>
+    <xacro:wheel_joint position="back_right" bot_center_to_wheel_center_x="${bot_center_to_wheel_center_x}" bot_center_to_wheel_center_y="${bot_center_to_wheel_center_y}"/>
+    <!-- BACK RIGHT WHEEL JOINT -->
+    <xacro:wheel position="back_right" radius="${wheel_radius}" thickness="${wheel_thickness}" mass="${wheel_mass}"/>
 </robot>

Commit message: Initial D435 Files Commit

File: description/robot_core.xacro (robot description, xacro)
@@ -30,4 +30,17 @@
     <link name="base_link">
     </link>
+    <xacro:arg name="use_nominal_extrinsics" default="false"/>
+    <xacro:arg name="add_plug" default="false" />
+    <xacro:arg name="use_mesh" default="true" />
+    <xacro:arg name="name" default="TEST435" />
+    <xacro:arg name="topics_ns" default="TEST435" />
+    <xacro:arg name="publish_pointcloud" default="false" />
+    <xacro:include filename="_d435.urdf.xacro" />
+    <xacro:sensor_d435 parent="base_link" use_nominal_extrinsics="$(arg use_nominal_extrinsics)" add_plug="$(arg add_plug)" use_mesh="$(arg use_mesh)" name="$(arg name)" topics_ns="$(arg topics_ns)" publish_pointcloud="$(arg publish_pointcloud)">
+      <origin xyz="0 0 1" rpy="0 0 0"/>
+    </xacro:sensor_d435>
+    <xacro:sensor_d435 name="test" topics_ns="test" parent="base_link" publish_pointcloud="true">
+        <origin xyz="0 0 0" rpy="0 0 0" />
+      </xacro:sensor_d435>
     <!-- CHASSIS -->
     <!-- Bottom plate .125" not included in robot model-->
