Commit message: Best attempt at d435 integration

File: description/_d435.urdf.xacro (robot description, xacro)
@@ -54,5 +54,5 @@
           <origin xyz="${d435_zero_depth_to_glass + d435_glass_to_front} ${-d435_cam_depth_py} 0" rpy="${M_PI/2} 0 ${M_PI/2}"/>
           <geometry>
-            <mesh filename="package://realsense2_description/meshes/d435.dae" />
+            <mesh filename="../meshes/d435.dae" />
           </geometry>
         </xacro:if>

File: description/_usb_plug.urdf.xacro (robot description, xacro)
@@ -20,5 +20,5 @@
         <geometry>
           <!--box size="0.044850 0.008 0.0185" /-->
-          <mesh filename="package://realsense2_description/meshes/plug.stl" />
+          <mesh filename="../meshes/plug.stl" />
         </geometry>
         <material name="plastic"/>
@@ -28,5 +28,5 @@
         <geometry>
           <!--box size="0.044850 0.008 0.0185" /-->
-          <mesh filename="package://realsense2_description/meshes/plug_collision.stl" />
+          <mesh filename="../meshes/plug_collision.stl" />
         </geometry>
       </collision>
